Commit message: add bullet

File: xtrainer_arm.urdf (robot description, URDF)
Before this commit: robot xtrainer_arm, 7 links, 6 joints
Links:
- link LINK_0: geometry collision mesh filename=meshes/base_link.STL; visual mesh filename=meshes/base_link.STL
- link LINK_1: geometry collision mesh filename=meshes/J1.STL; visual mesh filename=meshes/J1.STL
- link LINK_2: geometry collision mesh filename=meshes/J2.STL; visual mesh filename=meshes/J2.STL
- link LINK_3: geometry collision mesh filename=meshes/J3.STL; visual mesh filename=meshes/J3.STL
- link LINK_4: geometry collision mesh filename=meshes/J4.STL; visual mesh filename=meshes/J4.STL
- link LINK_5: geometry collision mesh filename=meshes/J5.STL; visual mesh filename=meshes/J5.STL
- link LINK_6: geometry collision mesh filename=meshes/J6.STL; visual mesh filename=meshes/J6.STL
